File: hardware/ESP32.kicad_sch (KiCad schematic)
At the start: 16 parts, among them J2 Conn_01x04, J3 Conn_01x05, U4 ESP32-C6-WROOM-1U-N4

Commit message: Update references from ESP32-S2 to ESP32-C6
Parts:
- U4: footprint ESP32_C6_WROOM_1U_N4 (1):XCVR_ESP32-C6-WROOM-1U-N4 -> ESP32_C6_WROOM_1U_N4:XCVR_ESP32-C6-WROOM-1U-N4
Changed lines of the file:
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@@
       (effects (font (size 1.27 1.27)))
     )
-    (property "Footprint" "ESP32_C6_WROOM_1U_N4 (1):XCVR_ESP32-C6-WROOM-1U-N4" (at 123.19 95.25 0)
+    (property "Footprint" "ESP32_C6_WROOM_1U_N4:XCVR_ESP32-C6-WROOM-1U-N4" (at 123.19 95.25 0)
       (effects (font (size 1.27 1.27)) (justify bottom) hide)
     )
