File: hardware/LanderControl.kicad_pcb (KiCad board)
At the start: 4 copper layers, 140 x 54 mm, 161 parts, among them J2 Conn_01x04, J3 Conn_01x05, J5 MEM2051-00-195-00-A, Q1 BC846, Q2 BC846, Q3 BC846, Q4 BC846, Q5 BC846, Q6 BC846, Q7 BC846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

Commit message: Replace PCA9500 I/O expander with TCA9534
Parts:
- U15: value PCA9500PW,118 -> TCA9534APWR
Changed lines of the file:
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@@
         (effects (font (size 1.640409 1.640409) (thickness 0.15)))
     )
-    (fp_text value "PCA9500PW,118" (at 14.276425 4.046255) (layer "F.Fab")
+    (fp_text value "TCA9534APWR" (at 14.276425 4.046255) (layer "F.Fab")
         (effects (font (size 1.64311 1.64311) (thickness 0.15)))
     )
